File: hardware/dawn.brd (EAGLE design)
At the start: 68.2 x 68.6 mm, 33 parts, among them IC1 ATMEGA168-20P, IC3 DS1307, Q2 16Mhz, Q3 32.768kHz, Q4 BUZ11BV, T3 BC547B, T4 BC547B, X1 MKDSN1,5/2-5,08, X2 MKDSN1,5/2-5,08

Commit message: Updated schematics and firmware for ATMEGA328P.
Parts:
- IC1: value ATMEGA168-20P -> ATMEGA328-20P; device adafruit:DIL28-3 -> atmega328:DIL28-3
Changed lines of the file:
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@@
 <element name="X1" library="con-phoenix-508" package="MKDSN1,5/2-5,08" value="MKDSN1,5/2-5,08" x="73.66" y="21.59"/>
 <element name="X2" library="con-phoenix-508" package="MKDSN1,5/2-5,08" value="MKDSN1,5/2-5,08" x="86.36" y="21.59"/>
-<element name="IC1" library="adafruit" package="DIL28-3" value="ATMEGA168-20P" x="49.53" y="45.72" rot="R270"/>
+<element name="IC1" library="atmega328" package="DIL28-3" value="ATMEGA328-20P" x="49.53" y="45.72" rot="R270"/>
 <element name="ISP1" library="adafruit" package="AVRISP" value="AVRISP-6" x="50.8" y="22.86" rot="R270"/>
 <element name="JP1" library="pinhead" package="1X05" value="GPIO" x="40.64" y="31.75" rot="R90"/>

Commit message: Cleanup
Parts:
- removed ISP1: AVRISP-6, adafruit:AVRISP
- added U$2: AVR-ISP, isp:AVR-ISP
- C6, C7: value 33pF -> 22pF
Connections:
- net +5V: now also U$2.VCC; no longer ISP1.2
- net GND: now also U$2.GND; no longer ISP1.6
- net N$2: now also U$2.MISO; no longer ISP1.1
- net N$3: now also U$2.SCK; no longer ISP1.3
- net N$4: now also U$2.RST; no longer ISP1.5
- net N$5: now also U$2.MOSI; no longer ISP1.4
Routing:
- net +5V: track 165.5 -> 166.8 mm
Changed lines of the file:
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@@
 </autorouter>
 <elements>
-<element name="C6" library="rcl" package="C050-025X075" value="33pF" x="43.18" y="41.91" rot="R90"/>
-<element name="C7" library="rcl" package="C025-025X050" value="33pF" x="40.64" y="43.18" rot="R90"/>
+<element name="C6" library="rcl" package="C050-025X075" value="22pF" x="43.18" y="41.91" rot="R90"/>
+<element name="C7" library="rcl" package="C025-025X050" value="22pF" x="40.64" y="43.18" rot="R90"/>
 <element name="C8" library="rcl" package="C025-025X050" value="100nF" x="55.88" y="45.72" rot="R90"/>
 <element name="C9" library="rcl" package="C025-025X050" value="100nF" x="41.91" y="46.99" rot="R180"/>
@@
 <element name="X2" library="con-phoenix-508" package="MKDSN1,5/2-5,08" value="MKDSN1,5/2-5,08" x="86.36" y="21.59"/>
 <element name="IC1" library="atmega328" package="DIL28-3" value="ATMEGA328-20P" x="49.53" y="45.72" rot="R270"/>
-<element name="ISP1" library="adafruit" package="AVRISP" value="AVRISP-6" x="50.8" y="22.86" rot="R270"/>
 <element name="JP1" library="pinhead" package="1X05" value="GPIO" x="40.64" y="31.75" rot="R90"/>
 <element name="KK1" library="heatsink" package="PF752" value="PF750" x="86.36" y="52.07"/>
@@
 <element name="C1" library="rcl" package="E5-6" value="100uF/35V" x="73.66" y="39.37" rot="R180"/>
 <element name="D1" library="diode" package="DO35Z10" value="SB140" x="76.2" y="34.29" rot="R180"/>
+<element name="U$2" library="isp" package="AVR-ISP" value="AVR-ISP" x="50.8" y="22.86" rot="R180"/>
 </elements>
 <signals>
@@
 <wire x1="38.1" y1="52.07" x2="43.18" y2="52.07" width="0.4064" layer="16"/>
 <wire x1="68.58" y1="64.77" x2="58.42" y2="64.77" width="0.4064" layer="16"/>
-<contactref element="ISP1" pad="2"/>
 <contactref element="IC1" pad="7"/>
 <contactref element="IC1" pad="21"/>
@@
 <wire x1="55.88" y1="64.77" x2="58.42" y2="64.77" width="0.4064" layer="16"/>
 <contactref element="X1" pad="2"/>
-<wire x1="53.34" y1="21.59" x2="68.58" y2="21.59" width="0.4064" layer="16"/>
 <via x="68.58" y="44.45" extent="1-16" drill="0.6" shape="square"/>
 <wire x1="68.58" y1="44.45" x2="58.42" y2="44.45" width="0.4064" layer="1"/>
@@
 <wire x1="86.36" y1="49.53" x2="86.36" y2="39.37" width="1.27" layer="16"/>
 <wire x1="86.36" y1="39.37" x2="76.2" y2="39.37" width="1.27" layer="16"/>
-<wire x1="68.58" y1="21.59" x2="68.58" y2="44.45" width="0.4064" layer="16"/>
+<wire x1="68.58" y1="21.59" x2="68.58" y2="22.86" width="0.4064" layer="16"/>
+<wire x1="68.58" y1="22.86" x2="68.58" y2="44.45" width="0.4064" layer="16"/>
 <wire x1="68.58" y1="44.45" x2="73.66" y2="44.45" width="0.4064" layer="16"/>
 <wire x1="73.66" y1="44.45" x2="73.66" y2="39.37" width="0.4064" layer="16"/>
 <wire x1="73.66" y1="39.37" x2="76.2" y2="39.37" width="0.4064" layer="16"/>
+<contactref element="U$2" pad="VCC"/>
+<wire x1="53.34" y1="21.59" x2="68.58" y2="21.59" width="0.4064" layer="16"/>
+<wire x1="68.58" y1="21.59" x2="68.58" y2="22.86" width="0.4064" layer="16"/>
 </signal>
 <signal name="GND">
@@
 <wire x1="71.12" y1="34.29" x2="71.12" y2="29.21" width="1.27" layer="16"/>
 <wire x1="71.12" y1="29.21" x2="71.12" y2="24.155" width="1.27" layer="16"/>
-<contactref element="ISP1" pad="6"/>
 <contactref element="IC1" pad="8"/>
 <contactref element="IC1" pad="22"/>
@@
 <wire x1="60.96" y1="74.93" x2="60.96" y2="67.31" width="0.4064" layer="16"/>
 <wire x1="60.96" y1="67.31" x2="50.8" y2="67.31" width="0.4064" layer="16"/>
-<wire x1="48.26" y1="21.59" x2="40.64" y2="21.59" width="0.4064" layer="16"/>
 <wire x1="40.64" y1="21.59" x2="40.64" y2="26.67" width="0.4064" layer="16"/>
 <wire x1="40.64" y1="26.67" x2="33.02" y2="26.67" width="0.4064" layer="16"/>
@@
 <wire x1="71.12" y1="39.37" x2="71.12" y2="41.91" width="0.4064" layer="16"/>
 <wire x1="55.88" y1="52.07" x2="60.96" y2="52.07" width="0.4064" layer="16"/>
+<contactref element="U$2" pad="GND"/>
+<wire x1="40.64" y1="21.59" x2="48.26" y2="21.59" width="0.4064" layer="16"/>
 </signal>
 <signal name="N$13">
@@
 <signal name="N$2">
 <contactref element="IC1" pad="18"/>
-<contactref element="ISP1" pad="1"/>
 <wire x1="53.34" y1="36.83" x2="60.96" y2="36.83" width="0.4064" layer="16"/>
 <wire x1="60.96" y1="36.83" x2="60.96" y2="24.13" width="0.4064" layer="16"/>
-<wire x1="60.96" y1="24.13" x2="53.34" y2="24.13" width="0.4064" layer="16"/>
+<contactref element="U$2" pad="MISO"/>
+<wire x1="53.34" y1="24.13" x2="60.96" y2="24.13" width="0.4064" layer="16"/>
 </signal>
 <signal name="N$3">
 <contactref element="IC1" pad="19"/>
-<contactref element="ISP1" pad="3"/>
 <wire x1="53.34" y1="39.37" x2="50.8" y2="39.37" width="0.4064" layer="16"/>
+<contactref element="U$2" pad="SCK"/>
 <wire x1="50.8" y1="39.37" x2="50.8" y2="24.13" width="0.4064" layer="16"/>
 </signal>
 <signal name="N$4">
-<contactref element="ISP1" pad="5"/>
 <contactref element="IC1" pad="1"/>
 <contactref element="R11" pad="2"/>
 <wire x1="43.18" y1="62.23" x2="45.72" y2="62.23" width="0.4064" layer="16"/>
 <wire x1="45.72" y1="62.23" x2="48.26" y2="62.23" width="0.4064" layer="16"/>
-<wire x1="48.26" y1="24.13" x2="48.26" y2="39.37" width="0.4064" layer="16"/>
 <wire x1="48.26" y1="39.37" x2="48.26" y2="40.64" width="0.4064" layer="16"/>
 <wire x1="48.26" y1="40.64" x2="48.26" y2="41.91" width="0.4064" layer="16"/>
@@
 <wire x1="48.26" y1="40.64" x2="48.26" y2="60.96" width="0.4064" layer="16"/>
 <wire x1="48.26" y1="60.96" x2="48.26" y2="62.23" width="0.4064" layer="16"/>
+<contactref element="U$2" pad="RST"/>
+<wire x1="48.26" y1="24.13" x2="48.26" y2="39.37" width="0.4064" layer="16"/>
 </signal>
 <signal name="N$5">
 <contactref element="IC1" pad="17"/>
-<contactref element="ISP1" pad="4"/>
 <wire x1="53.34" y1="34.29" x2="58.42" y2="34.29" width="0.4064" layer="16"/>
 <wire x1="58.42" y1="34.29" x2="58.42" y2="27.94" width="0.4064" layer="16"/>
@@
 <wire x1="58.42" y1="26.67" x2="58.42" y2="27.94" width="0.4064" layer="16"/>
 <wire x1="58.42" y1="27.94" x2="58.42" y2="26.67" width="0.4064" layer="16"/>
-<wire x1="50.8" y1="21.59" x2="50.8" y2="19.05" width="0.4064" layer="16"/>
 <wire x1="50.8" y1="19.05" x2="58.42" y2="19.05" width="0.4064" layer="16"/>
 <via x="58.42" y="19.05" extent="1-16" drill="0.6" shape="square"/>
@@
 <via x="58.42" y="26.67" extent="1-16" drill="0.6" shape="square"/>
 <wire x1="58.42" y1="26.67" x2="58.42" y2="27.94" width="0.4064" layer="16"/>
+<contactref element="U$2" pad="MOSI"/>
+<wire x1="50.8" y1="19.05" x2="50.8" y2="21.59" width="0.4064" layer="16"/>
 </signal>
 <signal name="N$1">

Commit message: Fixed.
Parts:
- R1: value 1k -> 470
- R2: value 10k -> 1k
Routing:
- net GND: track 223.5 -> 221.0 mm
Changed lines of the file:
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@@
 <element name="JP1" library="pinhead" package="1X05" value="GPIO" x="40.64" y="31.75" rot="R90"/>
 <element name="KK1" library="heatsink" package="PF752" value="PF750" x="86.36" y="52.07"/>
-<element name="R1" library="rcl" package="0204V" value="1k" x="55.88" y="50.8" rot="R90"/>
-<element name="R2" library="ptc-ntc" package="B57164" value="10k" x="58.42" y="46.99" rot="R270">
+<element name="R1" library="rcl" package="0204V" value="470" x="55.88" y="50.8" rot="R90"/>
+<element name="R2" library="ptc-ntc" package="B57164" value="1k" x="58.42" y="46.99" rot="R270">
 <attribute name="OC_NEWARK" value="29M3118" x="58.42" y="46.99" size="1.778" layer="27" rot="R270" display="off"/>
 <attribute name="MPN" value="B57164K474K52" x="58.42" y="46.99" size="1.778" layer="27" rot="R270" display="off"/>
@@
 <wire x1="45.72" y1="44.45" x2="43.18" y2="44.45" width="0.4064" layer="16"/>
 <wire x1="40.64" y1="44.45" x2="43.18" y2="44.45" width="0.4064" layer="16"/>
-<wire x1="40.64" y1="46.99" x2="38.1" y2="46.99" width="0.4064" layer="16"/>
-<wire x1="45.72" y1="44.45" x2="38.1" y2="44.45" width="0.4064" layer="16"/>
-<wire x1="38.1" y1="44.45" x2="38.1" y2="46.99" width="0.4064" layer="16"/>
+<wire x1="45.72" y1="44.45" x2="40.64" y2="44.45" width="0.4064" layer="16"/>
+<wire x1="40.64" y1="44.45" x2="40.64" y2="46.99" width="0.4064" layer="16"/>
 <wire x1="53.34" y1="46.99" x2="55.88" y2="46.99" width="0.4064" layer="16"/>
 <wire x1="55.88" y1="46.99" x2="60.96" y2="46.99" width="0.4064" layer="16"/>
@@
 <wire x1="40.64" y1="26.67" x2="33.02" y2="26.67" width="0.4064" layer="16"/>
 <wire x1="33.02" y1="26.67" x2="33.02" y2="46.99" width="0.4064" layer="16"/>
-<wire x1="38.1" y1="46.99" x2="33.02" y2="46.99" width="0.4064" layer="16"/>
+<wire x1="40.64" y1="46.99" x2="33.02" y2="46.99" width="0.4064" layer="16"/>
 <wire x1="33.02" y1="46.99" x2="33.02" y2="54.61" width="0.4064" layer="16"/>
 <wire x1="33.02" y1="54.61" x2="33.02" y2="67.31" width="0.4064" layer="16"/>

Commit message: Cleanup
Parts:
- removed R28: 1k, rcl:0204/5
- removed R29: 10k, rcl:0204V
- removed T4: BC547B, transistor-neu-to92:TO92-EBC
- moved R24 2.54 mm to (69.8, 49.5)
Connections:
- removed net N$43: R24.1, R29.2, T4.E
- net +5V: no longer T4.C
- net GND: no longer R28.1, R29.1
- net N$41: now also R24.1; no longer R28.2, T4.B
Routing:
- net N$43: track 5.08 -> 0.00 mm
- net N$37: track 12.7 -> 10.2 mm
Changed lines of the file:
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@@
 <element name="R13" library="rcl" package="0204V" value="10k" x="55.88" y="63.5" rot="R270"/>
 <element name="U$1" library="jy-mcu" package="JY-MCU" value="JY-MCU" x="38.1" y="55.88" rot="R180"/>
-<element name="R24" library="rcl" package="0204/7" value="10" x="69.85" y="52.07"/>
+<element name="R24" library="rcl" package="0204/7" value="10" x="69.85" y="49.53"/>
 <element name="Q4" library="transistor-power" package="TO220BV" value="BUZ11BV" x="86.36" y="52.07"/>
 <element name="R25" library="rcl" package="0411/12" value="1W" x="77.47" y="29.21"/>
@@
 <element name="C10" library="rcl" package="C025-025X050" value="100pF" x="64.77" y="34.29"/>
 <element name="R27" library="rcl" package="0207/10" value="4.7k" x="60.96" y="29.21"/>
-<element name="R28" library="rcl" package="0204/5" value="1k" x="63.5" y="46.99"/>
-<element name="T4" library="transistor-neu-to92" package="TO92-EBC" value="BC547B" x="66.04" y="50.8"/>
-<element name="R29" library="rcl" package="0204V" value="10k" x="62.23" y="52.07"/>
 <element name="X1" library="con-phoenix-508" package="MKDSN1,5/2-5,08" value="MKDSN1,5/2-5,08" x="73.66" y="21.59"/>
 <element name="X2" library="con-phoenix-508" package="MKDSN1,5/2-5,08" value="MKDSN1,5/2-5,08" x="86.36" y="21.59"/>
@@
 <contactref element="C9" pad="1"/>
 <contactref element="U$1" pad="VCC"/>
-<contactref element="T4" pad="C"/>
-<wire x1="68.58" y1="49.53" x2="68.58" y2="59.69" width="0.4064" layer="16"/>
 <wire x1="38.1" y1="52.07" x2="43.18" y2="52.07" width="0.4064" layer="16"/>
 <wire x1="68.58" y1="64.77" x2="58.42" y2="64.77" width="0.4064" layer="16"/>
@@
 <wire x1="76.1789" y1="21.615" x2="76.2" y2="21.615" width="1.27" layer="16"/>
 <wire x1="86.36" y1="49.53" x2="86.36" y2="44.45" width="1.27" layer="16"/>
-<wire x1="68.58" y1="49.53" x2="68.58" y2="44.45" width="0.4064" layer="16"/>
 <wire x1="86.36" y1="49.53" x2="86.36" y2="39.37" width="1.27" layer="16"/>
 <wire x1="86.36" y1="39.37" x2="76.2" y2="39.37" width="1.27" layer="16"/>
@@
 <wire x1="53.34" y1="21.59" x2="68.58" y2="21.59" width="0.4064" layer="16"/>
 <wire x1="68.58" y1="21.59" x2="68.58" y2="22.86" width="0.4064" layer="16"/>
+<wire x1="68.58" y1="44.45" x2="68.58" y2="59.69" width="0.4064" layer="16"/>
 </signal>
 <signal name="GND">
@@
 <contactref element="T3" pad="E"/>
 <contactref element="R25" pad="1"/>
-<contactref element="R28" pad="1"/>
-<contactref element="R29" pad="1"/>
 <wire x1="71.12" y1="34.29" x2="71.12" y2="29.21" width="1.27" layer="16"/>
 <wire x1="71.12" y1="29.21" x2="71.12" y2="24.155" width="1.27" layer="16"/>
@@
 <contactref element="IC1" pad="22"/>
 <contactref element="X1" pad="1"/>
-<wire x1="60.96" y1="41.91" x2="60.96" y2="46.99" width="0.4064" layer="16"/>
 <wire x1="71.0989" y1="21.615" x2="71.12" y2="24.155" width="1.27" layer="16"/>
 <wire x1="71.12" y1="24.155" x2="71.12" y2="24.13" width="1.27" layer="16"/>
@@
 <wire x1="60.96" y1="41.91" x2="71.12" y2="41.91" width="0.4064" layer="1"/>
 <via x="71.12" y="41.91" extent="1-16" drill="0.6" shape="square"/>
-<wire x1="60.96" y1="52.07" x2="60.96" y2="46.99" width="0.4064" layer="16"/>
 <wire x1="53.34" y1="46.99" x2="50.8" y2="46.99" width="0.4064" layer="16"/>
 <contactref element="JP1" pad="1"/>
@@
 <wire x1="40.64" y1="44.45" x2="40.64" y2="46.99" width="0.4064" layer="16"/>
 <wire x1="53.34" y1="46.99" x2="55.88" y2="46.99" width="0.4064" layer="16"/>
-<wire x1="55.88" y1="46.99" x2="60.96" y2="46.99" width="0.4064" layer="16"/>
 <wire x1="50.8" y1="46.99" x2="50.8" y2="67.31" width="0.4064" layer="16"/>
 <wire x1="50.8" y1="67.31" x2="33.02" y2="67.31" width="0.4064" layer="16"/>
@@
 <wire x1="71.12" y1="34.29" x2="71.12" y2="39.37" width="1.27" layer="16"/>
 <wire x1="71.12" y1="39.37" x2="71.12" y2="41.91" width="0.4064" layer="16"/>
-<wire x1="55.88" y1="52.07" x2="60.96" y2="52.07" width="0.4064" layer="16"/>
 <contactref element="U$2" pad="GND"/>
 <wire x1="40.64" y1="21.59" x2="48.26" y2="21.59" width="0.4064" layer="16"/>
+<wire x1="60.96" y1="41.91" x2="60.96" y2="46.99" width="0.4064" layer="16"/>
+<wire x1="60.96" y1="46.99" x2="55.88" y2="46.99" width="0.4064" layer="16"/>
+<wire x1="55.88" y1="52.07" x2="60.96" y2="52.07" width="0.4064" layer="16"/>
+<wire x1="60.96" y1="52.07" x2="60.96" y2="46.99" width="0.4064" layer="16"/>
 </signal>
 <signal name="N$13">
@@
 <contactref element="Q4" pad="G"/>
 <contactref element="R24" pad="2"/>
-<wire x1="83.82" y1="52.07" x2="73.66" y2="52.07" width="0.4064" layer="16"/>
-<wire x1="83.82" y1="49.53" x2="83.82" y2="52.07" width="0.4064" layer="16"/>
+<wire x1="83.82" y1="49.53" x2="73.66" y2="49.53" width="0.4064" layer="16"/>
 </signal>
 <signal name="N$39">
@@
 <contactref element="C10" pad="2"/>
 <contactref element="T3" pad="C"/>
-<contactref element="T4" pad="B"/>
-<contactref element="R28" pad="2"/>
 <contactref element="R27" pad="2"/>
-<wire x1="66.04" y1="49.53" x2="66.04" y2="46.99" width="0.4064" layer="16"/>
 <wire x1="66.04" y1="29.21" x2="66.04" y2="34.29" width="0.4064" layer="16"/>
 <wire x1="66.04" y1="39.37" x2="66.04" y2="34.29" width="0.4064" layer="16"/>
-<wire x1="66.04" y1="46.99" x2="66.04" y2="39.37" width="0.4064" layer="16"/>
-</signal>
-<signal name="N$43">
 <contactref element="R24" pad="1"/>
-<contactref element="R29" pad="2"/>
-<contactref element="T4" pad="E"/>
-<wire x1="63.5" y1="49.53" x2="63.5" y2="52.07" width="0.4064" layer="16"/>
-<wire x1="63.5" y1="52.07" x2="66.04" y2="52.07" width="0.4064" layer="16"/>
+<wire x1="66.04" y1="39.37" x2="66.04" y2="49.53" width="0.4064" layer="16"/>
 </signal>
 <signal name="N$2">

Commit message: Fixed minors.
Parts:
- added C2: 100nF, rcl:C025-025X050
Connections:
- removed net N$15: L1.2, X2.2
- new net N$16: Q4.D, X2.2
- net +5V: now also C2.1, D1.C, L1.1; no longer Q4.D
- net GND: now also C2.2
- net N$11: now also L1.2, X2.1; no longer D1.C, L1.1, Q4.S
- net N$39: now also Q4.S; no longer X2.1
Routing:
- net N$16: track 0.00 -> 45.7 mm
- net N$39: track 12.7 -> 33.0 mm
- net +5V: track 166.8 -> 152.8 mm
- net N$11: track 22.9 -> 12.7 mm
- net GND: track 221.0 -> 231.1 mm
- net N$15: track 7.66 -> 0.00 mm
Other:
- board text added: "Lampe rev. 2"
- board text removed: "Lampe rev. 1"
Changed lines of the file:
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@@
 <?xml version="1.0" encoding="utf-8"?>
 <!DOCTYPE eagle SYSTEM "eagle.dtd">
-<eagle version="7.1.0">
+<eagle version="7.5.0">
 <drawing>
 <settings>
@@
 <dimension x1="30.48" y1="80" x2="30.48" y2="11.43" x3="27.94" y3="45.715" textsize="1.778" layer="20"/>
 <dimension x1="30.48" y1="80" x2="99.06" y2="80.01" x3="64.76963125" y3="82.54519375" textsize="1.778" layer="20"/>
-<text x="40.64" y="72.39" size="1.778" layer="20">Lampe rev. 1</text>
+<text x="40.64" y="72.39" size="1.778" layer="20">Lampe rev. 2</text>
 <wire x1="83.82" y1="15.24" x2="85.09" y2="15.24" width="0.4064" layer="21"/>
 <wire x1="85.09" y1="16.51" x2="85.09" y2="13.97" width="0.4064" layer="21"/>
@@
 <element name="D1" library="diode" package="DO35Z10" value="SB140" x="76.2" y="34.29" rot="R180"/>
 <element name="U$2" library="isp" package="AVR-ISP" value="AVR-ISP" x="50.8" y="22.86" rot="R180"/>
+<element name="C2" library="rcl" package="C025-025X050" value="100nF" x="67.31" y="57.15" rot="R180"/>
 </elements>
 <signals>
@@
 <wire x1="53.34" y1="44.45" x2="55.88" y2="44.45" width="0.4064" layer="16"/>
 <contactref element="R2" pad="2"/>
-<contactref element="Q4" pad="D"/>
 <contactref element="C1" pad="+"/>
-<wire x1="76.2" y1="21.615" x2="76.2" y2="39.37" width="1.27" layer="16"/>
+<wire x1="76.2" y1="21.615" x2="76.2" y2="34.29" width="1.27" layer="16"/>
 <wire x1="76.1789" y1="21.615" x2="76.2" y2="21.615" width="1.27" layer="16"/>
-<wire x1="86.36" y1="49.53" x2="86.36" y2="44.45" width="1.27" layer="16"/>
-<wire x1="86.36" y1="49.53" x2="86.36" y2="39.37" width="1.27" layer="16"/>
-<wire x1="86.36" y1="39.37" x2="76.2" y2="39.37" width="1.27" layer="16"/>
-<wire x1="68.58" y1="21.59" x2="68.58" y2="22.86" width="0.4064" layer="16"/>
-<wire x1="68.58" y1="22.86" x2="68.58" y2="44.45" width="0.4064" layer="16"/>
+<wire x1="76.2" y1="34.29" x2="76.2" y2="39.37" width="1.27" layer="16"/>
+<wire x1="68.58" y1="21.59" x2="68.58" y2="44.45" width="0.4064" layer="16"/>
 <wire x1="68.58" y1="44.45" x2="73.66" y2="44.45" width="0.4064" layer="16"/>
 <wire x1="73.66" y1="44.45" x2="73.66" y2="39.37" width="0.4064" layer="16"/>
@@
 <contactref element="U$2" pad="VCC"/>
 <wire x1="53.34" y1="21.59" x2="68.58" y2="21.59" width="0.4064" layer="16"/>
-<wire x1="68.58" y1="21.59" x2="68.58" y2="22.86" width="0.4064" layer="16"/>
-<wire x1="68.58" y1="44.45" x2="68.58" y2="59.69" width="0.4064" layer="16"/>
+<wire x1="68.58" y1="44.45" x2="68.58" y2="57.15" width="0.4064" layer="16"/>
+<contactref element="D1" pad="C"/>
+<contactref element="L1" pad="1"/>
+<wire x1="68.58" y1="57.15" x2="68.58" y2="59.69" width="0.4064" layer="16"/>
+<wire x1="88.9" y1="34.29" x2="88.9" y2="34.25" width="1.27" layer="16"/>
+<wire x1="81.28" y1="34.29" x2="88.9" y2="34.29" width="1.27" layer="16"/>
+<wire x1="76.2" y1="34.29" x2="81.28" y2="34.29" width="1.27" layer="16"/>
+<contactref element="C2" pad="1"/>
 </signal>
 <signal name="GND">
@@
 <wire x1="55.88" y1="52.07" x2="60.96" y2="52.07" width="0.4064" layer="16"/>
 <wire x1="60.96" y1="52.07" x2="60.96" y2="46.99" width="0.4064" layer="16"/>
+<contactref element="C2" pad="2"/>
+<wire x1="66.04" y1="57.15" x2="66.04" y2="52.07" width="0.3048" layer="16"/>
+<wire x1="66.04" y1="52.07" x2="60.96" y2="52.07" width="0.3048" layer="16"/>
 </signal>
 <signal name="N$13">
@@
 <contactref element="R25" pad="2"/>
 <contactref element="R26" pad="1"/>
-<contactref element="X2" pad="1"/>
 <wire x1="81.28" y1="31.75" x2="83.82" y2="31.75" width="0.4064" layer="16"/>
-<wire x1="83.7989" y1="21.615" x2="83.82" y2="21.615" width="1.27" layer="16"/>
-<wire x1="83.82" y1="21.615" x2="83.82" y2="29.21" width="1.27" layer="16"/>
-<wire x1="83.82" y1="31.75" x2="83.82" y2="29.21" width="0.4064" layer="16"/>
+<contactref element="Q4" pad="S"/>
+<wire x1="88.9" y1="49.53" x2="91.44" y2="49.53" width="1.27" layer="16"/>
+<wire x1="91.44" y1="49.53" x2="91.44" y2="31.75" width="1.27" layer="16"/>
+<wire x1="91.44" y1="31.75" x2="83.82" y2="31.75" width="1.27" layer="16"/>
+<wire x1="83.82" y1="29.21" x2="83.82" y2="31.75" width="1.27" layer="16"/>
 </signal>
 <signal name="N$40">
@@
 <wire x1="55.88" y1="49.53" x2="58.42" y2="49.53" width="0.4064" layer="16"/>
 </signal>
+<signal name="N$16">
+<contactref element="Q4" pad="D"/>
+<contactref element="X2" pad="2"/>
+<wire x1="88.8789" y1="21.615" x2="93.98" y2="21.615" width="1.27" layer="16"/>
+<wire x1="93.98" y1="21.615" x2="93.98" y2="21.59" width="1.27" layer="16"/>
+<wire x1="93.98" y1="21.615" x2="93.98" y2="52.07" width="1.27" layer="16"/>
+<wire x1="93.98" y1="52.07" x2="86.36" y2="52.07" width="1.27" layer="16"/>
+<wire x1="86.36" y1="52.07" x2="86.36" y2="49.53" width="1.27" layer="16"/>
+</signal>
 <signal name="N$11">
-<contactref element="Q4" pad="S"/>
-<contactref element="D1" pad="C"/>
-<contactref element="L1" pad="1"/>
-<wire x1="88.9" y1="49.53" x2="88.9" y2="34.29" width="1.27" layer="16"/>
-<wire x1="88.9" y1="34.29" x2="88.9" y2="34.25" width="1.27" layer="16"/>
-<wire x1="81.28" y1="34.29" x2="88.9" y2="34.29" width="1.27" layer="16"/>
-</signal>
-<signal name="N$15">
 <contactref element="L1" pad="2"/>
-<contactref element="X2" pad="2"/>
-<wire x1="88.8789" y1="21.615" x2="88.9" y2="21.615" width="1.27" layer="16"/>
-<wire x1="88.9" y1="21.615" x2="88.9" y2="29.21" width="1.27" layer="16"/>
-<wire x1="88.9" y1="29.21" x2="88.9" y2="29.25" width="1.27" layer="16"/>
+<contactref element="X2" pad="1"/>
+<wire x1="88.9" y1="29.25" x2="88.9" y2="26.71" width="1.27" layer="16"/>
+<wire x1="88.9" y1="26.71" x2="83.82" y2="26.67" width="1.27" layer="16"/>
+<wire x1="83.82" y1="26.67" x2="83.7989" y2="21.59" width="1.27" layer="16"/>
+<wire x1="83.7989" y1="21.59" x2="83.7989" y2="21.615" width="1.27" layer="16"/>
 </signal>
 </signals>
