File: hardware/lampe.sch (EAGLE design)
At the start: 30 parts, among them IC1 ATMEGA168-20P, IC3 DS1307, Q2 16Mhz, Q3 32.768kHz, Q4 BUZ11BV, T3 BC547B, T4 BC547B, X1 MKDSN1,5/2-5,08, X2 MKDSN1,5/2-5,08

Commit message: Fixed.
Other:
- note added: "3V"
Changed lines of the file:
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@@
 <text x="134.62" y="-5.08" size="1.778" layer="91">2.9V @ 700mA, 240lm
 conrad: 182695</text>
-<text x="101.6" y="-12.7" size="1.778" layer="91">18K/W, TO-220
+<text x="99.06" y="-12.7" size="1.778" layer="91">18K/W, TO-220
 conrad: 183971</text>
+<text x="86.36" y="-12.7" size="1.778" layer="91">3V</text>
 </plain>
 <instances>
