File: hardware/lampe.brd (EAGLE design)
At the start: 68.2 x 68.6 mm, 33 parts, among them IC1 ATMEGA168-20P, IC3 DS1307, Q2 16Mhz, Q3 32.768kHz, Q4 BUZ11BV, T3 BC547B, T4 BC547B, X1 MKDSN1,5/2-5,08, X2 MKDSN1,5/2-5,08

Commit message: Minors.
Parts:
- moved C10 2.54 mm to (64.8, 34.3)
Routing:
- net N$40: track 10.2 -> 12.7 mm
Changed lines of the file:
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@@
 <?xml version="1.0" encoding="utf-8"?>
 <!DOCTYPE eagle SYSTEM "eagle.dtd">
-<eagle version="7.2.0">
+<eagle version="7.1.0">
 <drawing>
 <settings>
@@
 <element name="R26" library="rcl" package="0207/17" value="560" x="72.39" y="31.75" rot="R180"/>
 <element name="T3" library="transistor-neu-to92" package="TO92-EBC" value="BC547B" x="63.5" y="40.64"/>
-<element name="C10" library="rcl" package="C025-025X050" value="100pF" x="64.77" y="36.83"/>
+<element name="C10" library="rcl" package="C025-025X050" value="100pF" x="64.77" y="34.29"/>
 <element name="R27" library="rcl" package="0207/10" value="4.7k" x="60.96" y="29.21"/>
 <element name="R28" library="rcl" package="0204/5" value="1k" x="63.5" y="46.99"/>
@@
 <contactref element="C10" pad="1"/>
 <wire x1="63.5" y1="31.75" x2="63.5" y2="39.37" width="0.4064" layer="16"/>
-<wire x1="63.5" y1="39.37" x2="63.5" y2="36.83" width="0.4064" layer="16"/>
+<wire x1="63.5" y1="39.37" x2="63.5" y2="34.29" width="0.4064" layer="16"/>
 </signal>
 <signal name="N$41">
@@
 <contactref element="R27" pad="2"/>
 <wire x1="66.04" y1="49.53" x2="66.04" y2="46.99" width="0.4064" layer="16"/>
-<wire x1="66.04" y1="29.21" x2="66.04" y2="36.83" width="0.4064" layer="16"/>
-<wire x1="66.04" y1="39.37" x2="66.04" y2="36.83" width="0.4064" layer="16"/>
+<wire x1="66.04" y1="29.21" x2="66.04" y2="34.29" width="0.4064" layer="16"/>
+<wire x1="66.04" y1="39.37" x2="66.04" y2="34.29" width="0.4064" layer="16"/>
 <wire x1="66.04" y1="46.99" x2="66.04" y2="39.37" width="0.4064" layer="16"/>
 </signal>
